File: Kicad/speedometer_Arduino_Nano/speedometer_Arduino_Nano.kicad_sch (KiCad schematic)
At the start: 13 parts, among them J1 Conn_01x02_Socket, J2 Sensor Module 1, J3 Conn_01x02_Socket, J5 Sensor Module 2, M1 Tacho

Commit message: erweiterung Readme.md code
Parts:
- added D2, D3: LED, symbol Device:LED
- added LS1: Speaker, symbol Device:Speaker
- added R5, R6, R7: 220, Resistor_THT:R_Axial_DIN0207_L6.3mm_D2.5mm_P10.16mm_Horizontal, symbol Device:R
- added SW1: SW_DIP_x04, symbol Switch:SW_DIP_x04
Connections:
- net GND: now also D2.1 (K), D3.1 (K), LS1.2, SW1.1, SW1.2, SW1.3, SW1.4
- net LED-S2: now reaches A1.10 (D7)
- net LED-S2: now also R6.1
- net SP: now reaches A1.11 (D8)
- net SP: now also R7.1
- net sw1: now reaches A1.13 (D10)
- net sw1: now also SW1.8
- net sw2: now reaches A1.14 (D11)
- net sw2: now also SW1.7
- net sw3: now reaches A1.15 (D12)
- net sw3: now also SW1.6
- net sw4: now reaches A1.16 (D13)
- net sw4: now also SW1.5
- net LED-S1: now reaches A1.9 (D6)
- net LED-S1: now also R5.1
- net Power renamed +5V
- new net: D2.2 (A), R5.2
- new net: LS1.1, R7.2
- new net: D3.2 (A), R6.2
Other:
- note added: "Sensor LED Display"
- note added: "Servo Acceleration"
- note added: "Speaker"
- moved on the sheet: BT1, C1, D1, J2, J5, M1, R1, R2, R3, R4
